Commit message: Moveit & gazebo functionality

File: src/fairino3_v6_moveit2_config/config/fairino3_v6_robot.ros2_control.xacro (robot description, xacro)
@@ -3,52 +3,101 @@
     <xacro:macro name="fairino3_v6_robot_ros2_control" params="name initial_positions_file">
         <xacro:property name="initial_positions" value="${load_yaml(initial_positions_file)['initial_positions']}"/>
-        <ros2_control name="GazeboSimSystem" type="system">
-            <hardware>
-                <!-- By default, set up controllers for simulation. This won't work on real hardware -->
-                <plugin>gz_ros2_control/GazeboSimSystem</plugin>
-            </hardware>
-            <joint name="j1">
-                <command_interface name="position"/>
-                <state_interface name="position">
-                  <param name="initial_value">${initial_positions['j1']}</param>
-                </state_interface>
-            </joint>
-            <joint name="j2">
-                <command_interface name="position"/>
-                <state_interface name="position">
-                  <param name="initial_value">${initial_positions['j2']}</param>
-                </state_interface>
-            </joint>
-            <joint name="j3">
-                <command_interface name="position"/>
-                <state_interface name="position">
-                  <param name="initial_value">${initial_positions['j3']}</param>
-                </state_interface>
-            </joint>
-            <joint name="j4">
-                <command_interface name="position"/>
-                <state_interface name="position">
-                  <param name="initial_value">${initial_positions['j4']}</param>
-                </state_interface>
-            </joint>
-            <joint name="j5">
-                <command_interface name="position"/>
-                <state_interface name="position">
-                  <param name="initial_value">${initial_positions['j5']}</param>
-                </state_interface>
-            </joint>
-            <joint name="j6">
-                <command_interface name="position"/>
-                <state_interface name="position">
-                  <param name="initial_value">${initial_positions['j6']}</param>
-                </state_interface>
-            </joint>
-        </ros2_control>
-        <gazebo>
-            <plugin filename="libign_ros2_control-system.so"
-            name="gz_ros2_control::GazeboSimROS2ControlPlugin">
-                <parameters>$(find fairino3_v6_moveit2_config)/config/ros2_controllers.yaml</parameters>
-            </plugin>
-        </gazebo>
+        <!-- Xacro arg for control system (Defualted to Rviz/Moveit-->
+        <xacro:arg name="control_system" default="moveit"/>
+        <xacro:if value="${'$(arg control_system)' == 'moveit'}">
+            <ros2_control name="${name}" type="system">
+                <hardware>
+                    <!-- By default, set up controllers for simulation. This won't work on real hardware -->
+                    <plugin>fairino_hardware/FairinoHardwareInterface</plugin>
+                </hardware>
+                <joint name="j1">
+                    <command_interface name="position"/>
+                    <state_interface name="position">
+                      <param name="initial_value">${initial_positions['j1']}</param>
+                    </state_interface>
+                </joint>
+                <joint name="j2">
+                    <command_interface name="position"/>
+                    <state_interface name="position">
+                      <param name="initial_value">${initial_positions['j2']}</param>
+                    </state_interface>
+                </joint>
+                <joint name="j3">
+                    <command_interface name="position"/>
+                    <state_interface name="position">
+                      <param name="initial_value">${initial_positions['j3']}</param>
+                    </state_interface>
+                </joint>
+                <joint name="j4">
+                    <command_interface name="position"/>
+                    <state_interface name="position">
+                      <param name="initial_value">${initial_positions['j4']}</param>
+                    </state_interface>
+                </joint>
+                <joint name="j5">
+                    <command_interface name="position"/>
+                    <state_interface name="position">
+                      <param name="initial_value">${initial_positions['j5']}</param>
+                    </state_interface>
+                </joint>
+                <joint name="j6">
+                    <command_interface name="position"/>
+                    <state_interface name="position">
+                      <param name="initial_value">${initial_positions['j6']}</param>
+                    </state_interface>
+                </joint>
+            </ros2_control>
+        </xacro:if>
+        <!-- Gazebo Control system-->
+        <xacro:if value="${'$(arg control_system)' == 'gazebo'}">
+            <ros2_control name="GazeboSimSystem" type="system">
+                <hardware>
+                    <!-- Gazebo Simulation control -->
+                    <plugin>gz_ros2_control/GazeboSimSystem</plugin>
+                </hardware>
+                <joint name="j1">
+                    <command_interface name="position"/>
+                    <state_interface name="position">
+                      <param name="initial_value">${initial_positions['j1']}</param>
+                    </state_interface>
+                </joint>
+                <joint name="j2">
+                    <command_interface name="position"/>
+                    <state_interface name="position">
+                      <param name="initial_value">${initial_positions['j2']}</param>
+                    </state_interface>
+                </joint>
+                <joint name="j3">
+                    <command_interface name="position"/>
+                    <state_interface name="position">
+                      <param name="initial_value">${initial_positions['j3']}</param>
+                    </state_interface>
+                </joint>
+                <joint name="j4">
+                    <command_interface name="position"/>
+                    <state_interface name="position">
+                      <param name="initial_value">${initial_positions['j4']}</param>
+                    </state_interface>
+                </joint>
+                <joint name="j5">
+                    <command_interface name="position"/>
+                    <state_interface name="position">
+                      <param name="initial_value">${initial_positions['j5']}</param>
+                    </state_interface>
+                </joint>
+                <joint name="j6">
+                    <command_interface name="position"/>
+                    <state_interface name="position">
+                      <param name="initial_value">${initial_positions['j6']}</param>
+                    </state_interface>
+                </joint>
+            </ros2_control>
+            <gazebo>
+                <plugin filename="libign_ros2_control-system.so"
+                name="gz_ros2_control::GazeboSimROS2ControlPlugin">
+                    <parameters>$(find fairino3_v6_moveit2_config)/config/ros2_controllers.yaml</parameters>
+                </plugin>
+            </gazebo>
+        </xacro:if>
     </xacro:macro>
 </robot>

File: src/fairino3_v6_moveit2_config/config/fairino3_v6_robot.urdf.xacro (robot description, xacro)
@@ -8,7 +8,43 @@
     <xacro:fairino3_v6_robot_ros2_control name="FakeSystem" initial_positions_file="$(arg initial_positions_file)"/>
     <!-- Custom args -->
-    <xacro:arg name="gripper" default="None"/>
-<!--
-    <xacro:if value="$($(arg gripper) == 'pgc140')">
+    <!-- <xacro:arg name="gripper" default="None"/>
+    <xacro:arg name="mount" default='None'/> -->
+<!--     <xacro:if value="${$(arg gripper) == 'pgc140'}">
+        <link name="world_link">
+            <parent link="world"/>
+            <child
+        </link>
+    </xacro:if> -->
+    <!-- <xacro:if value="${$(arg mount) == 'box'}">
+        <link name="mount_link">
+            <joint name="fixed" type="fixed">
+                <parent link="mount_link"/>
+                <child link="world"/>
+            </joint>
+            <visual>
+                <geometry>
+                    <box size="1 1 1"/>
+                </geometry>
+                <material name="red">
+                    <color rgba="1 0 0 1"/>
+                </material>
+            </visual>
+            <collision>
+                <geometry>
+                    <box size="1 1 1"/>
+                </geometry>
+            </collision>
+            <inertial>
+                <mass value="1.0"/>
+                <inertia ixx="0.01" ixy="0.0" ixz="0.0" iyy="0.01" iyz="0.0" izz="0.01"/>
+            </inertial>
+        </link>
+    </xacro:if> -->
+    <!-- <xacro:if value="${$(arg mount) == 'None'}">
+        <link name="world"/>
+            <joint name="fixed" type="fixed">
+                <parent link="world"/>
+                <child link="base_link"/>
+            </joint>
     </xacro:if> -->
 </robot>
