Commit message: FR5 working, starting port of full robot catalog

File: src/fairino5_v6_moveit2_config/config/fairino5_v6_robot.ros2_control.xacro (robot description, xacro)
@@ -3,46 +3,101 @@
     <xacro:macro name="fairino5_v6_robot_ros2_control" params="name initial_positions_file">
         <xacro:property name="initial_positions" value="${load_yaml(initial_positions_file)['initial_positions']}"/>
-        <ros2_control name="${name}" type="system">
-            <hardware>
-                <!-- By default, set up controllers for simulation. This won't work on real hardware -->
-                <plugin>mock_components/GenericSystem</plugin>
-            </hardware>
-            <joint name="j1">
-                <command_interface name="position"/>
-                <state_interface name="position">
-                  <param name="initial_value">${initial_positions['j1']}</param>
-                </state_interface>
-            </joint>
-            <joint name="j2">
-                <command_interface name="position"/>
-                <state_interface name="position">
-                  <param name="initial_value">${initial_positions['j2']}</param>
-                </state_interface>
-            </joint>
-            <joint name="j3">
-                <command_interface name="position"/>
-                <state_interface name="position">
-                  <param name="initial_value">${initial_positions['j3']}</param>
-                </state_interface>
-            </joint>
-            <joint name="j4">
-                <command_interface name="position"/>
-                <state_interface name="position">
-                  <param name="initial_value">${initial_positions['j4']}</param>
-                </state_interface>
-            </joint>
-            <joint name="j5">
-                <command_interface name="position"/>
-                <state_interface name="position">
-                  <param name="initial_value">${initial_positions['j5']}</param>
-                </state_interface>
-            </joint>
-            <joint name="j6">
-                <command_interface name="position"/>
-                <state_interface name="position">
-                  <param name="initial_value">${initial_positions['j6']}</param>
-                </state_interface>
-            </joint>
-        </ros2_control>
+        <!-- Xacro arg for control system (Defualted to Rviz/Moveit-->
+        <xacro:arg name="control_system" default="moveit"/>
+        <xacro:if value="${'$(arg control_system)' == 'moveit'}">
+            <ros2_control name="${name}" type="system">
+                <hardware>
+                    <!-- By default, set up controllers for simulation. This won't work on real hardware -->
+                    <plugin>fairino_hardware/FairinoHardwareInterface</plugin>
+                </hardware>
+                <joint name="j1">
+                    <command_interface name="position"/>
+                    <state_interface name="position">
+                      <param name="initial_value">${initial_positions['j1']}</param>
+                    </state_interface>
+                </joint>
+                <joint name="j2">
+                    <command_interface name="position"/>
+                    <state_interface name="position">
+                      <param name="initial_value">${initial_positions['j2']}</param>
+                    </state_interface>
+                </joint>
+                <joint name="j3">
+                    <command_interface name="position"/>
+                    <state_interface name="position">
+                      <param name="initial_value">${initial_positions['j3']}</param>
+                    </state_interface>
+                </joint>
+                <joint name="j4">
+                    <command_interface name="position"/>
+                    <state_interface name="position">
+                      <param name="initial_value">${initial_positions['j4']}</param>
+                    </state_interface>
+                </joint>
+                <joint name="j5">
+                    <command_interface name="position"/>
+                    <state_interface name="position">
+                      <param name="initial_value">${initial_positions['j5']}</param>
+                    </state_interface>
+                </joint>
+                <joint name="j6">
+                    <command_interface name="position"/>
+                    <state_interface name="position">
+                      <param name="initial_value">${initial_positions['j6']}</param>
+                    </state_interface>
+                </joint>
+            </ros2_control>
+        </xacro:if>
+        <!-- Gazebo Control system-->
+        <xacro:if value="${'$(arg control_system)' == 'gazebo'}">
+            <ros2_control name="GazeboSimSystem" type="system">
+                <hardware>
+                    <!-- Gazebo Simulation control -->
+                    <plugin>gz_ros2_control/GazeboSimSystem</plugin>
+                </hardware>
+                <joint name="j1">
+                    <command_interface name="position"/>
+                    <state_interface name="position">
+                      <param name="initial_value">${initial_positions['j1']}</param>
+                    </state_interface>
+                </joint>
+                <joint name="j2">
+                    <command_interface name="position"/>
+                    <state_interface name="position">
+                      <param name="initial_value">${initial_positions['j2']}</param>
+                    </state_interface>
+                </joint>
+                <joint name="j3">
+                    <command_interface name="position"/>
+                    <state_interface name="position">
+                      <param name="initial_value">${initial_positions['j3']}</param>
+                    </state_interface>
+                </joint>
+                <joint name="j4">
+                    <command_interface name="position"/>
+                    <state_interface name="position">
+                      <param name="initial_value">${initial_positions['j4']}</param>
+                    </state_interface>
+                </joint>
+                <joint name="j5">
+                    <command_interface name="position"/>
+                    <state_interface name="position">
+                      <param name="initial_value">${initial_positions['j5']}</param>
+                    </state_interface>
+                </joint>
+                <joint name="j6">
+                    <command_interface name="position"/>
+                    <state_interface name="position">
+                      <param name="initial_value">${initial_positions['j6']}</param>
+                    </state_interface>
+                </joint>
+            </ros2_control>
+            <gazebo>
+                <plugin filename="libign_ros2_control-system.so"
+                name="gz_ros2_control::GazeboSimROS2ControlPlugin">
+                    <parameters>$(find fairino5_v6_moveit2_config)/config/ros2_controllers.yaml</parameters>
+                </plugin>
+            </gazebo>
+        </xacro:if>
     </xacro:macro>
 </robot>

File: src/fairino_description/urdf/fairino5_v6.urdf (robot description, URDF)
Before this commit: robot fairino5_v6_robot, 7 links, 6 joints
Links:
- added link world
Joints:
- added joint fixed: type fixed, parent world, child base_link
