Commit message: fr10 done

File: src/fairino_description/urdf/fairino10_v6.urdf (robot description, URDF)
Before this commit: robot fairino10_v6_robot, 7 links, 6 joints
Links:
- added link world
Joints:
- added joint fixed: type fixed, parent world, child base_link
- joint j1: limit lower=-3.0543 upper=3.0543 effort=150 velocity=3.15 -> lower=-3.0543 upper=3.0543 effort=250 velocity=3.15
- joint j2: limit lower=-4.6251 upper=1.4835 effort=150 velocity=3.15 -> lower=-4.6251 upper=1.4835 effort=250 velocity=3.15
- joint j3: limit lower=-2.8274 upper=2.8274 effort=150 velocity=3.15 -> lower=-2.8274 upper=2.8274 effort=250 velocity=3.15

File: src/fairino_description/urdf/fairino16_v6.urdf (robot description, URDF)
Before this commit: robot fairino16_v6_robot, 7 links, 6 joints
Links:
- added link world
Joints:
- added joint fixed: type fixed, parent world, child base_link

File: src/fairino_description/urdf/fairino20_v6.urdf (robot description, URDF)
Before this commit: robot fairino20_v6_robot, 7 links, 6 joints
Links:
- added link world
Joints:
- added joint fixed: type fixed, parent world, child base_link

File: src/fairino_description/urdf/fairino30_v6.urdf (robot description, URDF)
Before this commit: robot fairino30_v6_robot, 7 links, 6 joints
Links:
- added link world
Joints:
- added joint fixed: type fixed, parent world, child base_link

File: src/fairino_description/urdf/fairino3_mt_v6.urdf (robot description, URDF)
Before this commit: robot fairino3mt_v6_robot, 7 links, 6 joints
Links:
- added link world
Joints:
- added joint fixed: type fixed, parent world, child base_link

Commit message: Waiting on confirmation of 'effort' value in URDF

File: src/fairino_description/urdf/fairino10_v6.urdf (robot description, URDF)
Before this commit: robot fairino10_v6_robot, 8 links, 7 joints
Joints:
- joint j1: limit lower=-3.0543 upper=3.0543 effort=250 velocity=3.15 -> lower=-3.0543 upper=3.0543 effort=150 velocity=3.15
- joint j2: limit lower=-4.6251 upper=1.4835 effort=250 velocity=3.15 -> lower=-4.6251 upper=1.4835 effort=150 velocity=3.15
- joint j3: limit lower=-2.8274 upper=2.8274 effort=250 velocity=3.15 -> lower=-2.8274 upper=2.8274 effort=150 velocity=3.15

Commit message: all robot models added

File: src/fairino_description/urdf/fairino10_v6.urdf (robot description, URDF)
Before this commit: robot fairino10_v6_robot, 8 links, 7 joints
Joints:
- joint j1: limit lower=-3.0543 upper=3.0543 effort=150 velocity=3.15 -> lower=-3.0543 upper=3.0543 effort=330 velocity=3.15
- joint j2: limit lower=-4.6251 upper=1.4835 effort=150 velocity=3.15 -> lower=-4.6251 upper=1.4835 effort=330 velocity=3.15
- joint j4: limit lower=-4.6251 upper=1.4835 effort=28 velocity=3.2 -> lower=-4.6251 upper=1.4835 effort=54 velocity=3.2
- joint j5: limit lower=-3.0543 upper=3.0543 effort=28 velocity=3.2 -> lower=-3.0543 upper=3.0543 effort=54 velocity=3.2
- joint j6: limit lower=-3.0543 upper=3.0543 effort=28 velocity=3.2 -> lower=-3.0543 upper=3.0543 effort=54 velocity=3.2

File: src/fairino_description/urdf/fairino16_v6.urdf (robot description, URDF)
Before this commit: robot fairino16_v6_robot, 8 links, 7 joints
Joints:
- joint j1: limit lower=-3.0543 upper=3.0543 effort=150 velocity=3.15 -> lower=-3.0543 upper=3.0543 effort=330 velocity=3.15
- joint j2: limit lower=-4.6251 upper=1.4835 effort=150 velocity=3.15 -> lower=-4.6251 upper=1.4835 effort=330 velocity=3.15
- joint j4: limit lower=-4.6251 upper=1.4835 effort=28 velocity=3.2 -> lower=-4.6251 upper=1.4835 effort=54 velocity=3.2
- joint j5: limit lower=-3.0543 upper=3.0543 effort=28 velocity=3.2 -> lower=-3.0543 upper=3.0543 effort=54 velocity=3.2
- joint j6: limit lower=-3.0543 upper=3.0543 effort=28 velocity=3.2 -> lower=-3.0543 upper=3.0543 effort=54 velocity=3.2

File: src/fairino_description/urdf/fairino20_v6.urdf (robot description, URDF)
Before this commit: robot fairino20_v6_robot, 8 links, 7 joints
Joints:
- joint j1: limit lower=-3.0543 upper=3.0543 effort=150 velocity=3.15 -> lower=-3.0543 upper=3.0543 effort=738 velocity=3.15
- joint j2: limit lower=-4.6251 upper=1.4835 effort=150 velocity=3.15 -> lower=-4.6251 upper=1.4835 effort=738 velocity=3.15
- joint j3: limit lower=-2.8274 upper=2.8274 effort=150 velocity=3.15 -> lower=-2.8274 upper=2.8274 effort=433 velocity=3.15
- joint j4: limit lower=-4.6251 upper=1.4835 effort=28 velocity=3.2 -> lower=-4.6251 upper=1.4835 effort=107 velocity=3.2
- joint j5: limit lower=-3.0543 upper=3.0543 effort=28 velocity=3.2 -> lower=-3.0543 upper=3.0543 effort=107 velocity=3.2
- joint j6: limit lower=-3.0543 upper=3.0543 effort=28 velocity=3.2 -> lower=-3.0543 upper=3.0543 effort=107 velocity=3.2

File: src/fairino_description/urdf/fairino30_v6.urdf (robot description, URDF)
Before this commit: robot fairino30_v6_robot, 8 links, 7 joints
Joints:
- joint j1: limit lower=-3.0543 upper=3.0543 effort=150 velocity=3.15 -> lower=-3.0543 upper=3.0543 effort=738 velocity=3.15
- joint j2: limit lower=-4.6251 upper=1.4835 effort=150 velocity=3.15 -> lower=-4.6251 upper=1.4835 effort=738 velocity=3.15
- joint j3: limit lower=-2.8274 upper=2.8274 effort=150 velocity=3.15 -> lower=-2.8274 upper=2.8274 effort=433 velocity=3.15
- joint j4: limit lower=-4.6251 upper=1.4835 effort=28 velocity=3.2 -> lower=-4.6251 upper=1.4835 effort=107 velocity=3.2
- joint j5: limit lower=-3.0543 upper=3.0543 effort=28 velocity=3.2 -> lower=-3.0543 upper=3.0543 effort=107 velocity=3.2
- joint j6: limit lower=-3.0543 upper=3.0543 effort=28 velocity=3.2 -> lower=-3.0543 upper=3.0543 effort=107 velocity=3.2
